Commit message: Working on RViz Movement

File: src/car_model/urdf/carModel.urdf (robot description, URDF)
Before this commit: robot car_model, 7 links, 6 joints
Joints:
- joint back_left_wheel_to_back_axle: limit lower=3.14 upper=3.14 effort=1000.0 velocity=1.0 -> lower=-3140.0 upper=3140.0 effort=1000.0 velocity=1.0
- joint back_right_wheel_to_back_axle: limit lower=-3.14 upper=3.14 effort=1000.0 velocity=1.0 -> lower=-3140.0 upper=3140.0 effort=1000.0 velocity=1.0

File: src/car_model/urdf/carModel.xacro (robot description, xacro)
@@ -25,5 +25,5 @@
         <xacro:macro name="global_joint" params="child">
                 <joint name="world_joint_to_${child}" type="fixed">
-                        <parent link="base_link" />
+                        <parent link="world" />
                         <child link="${child}" />
                 </joint>
@@ -41,6 +41,6 @@
                                 <geometry>
                                         <box size="${baselength/2} ${baselength} ${baselength/8}" />
-                                        <origin rpy="0 0 0" xyz="0 0 ${baseheight}" />
                                 </geometry>
+                                <origin rpy="0 0 0" xyz="0 0 ${baseheight}" />
                         </collision>
                         <xacro:default_inertial mass="5"/>
@@ -130,6 +130,6 @@
         <xacro:car_front_wheel leftright="left" lr="${(axlelength/2) + 0.05}" axle="1" position="1" upper="0.785" lower="-0.393" />
         <xacro:car_front_wheel leftright="right" lr="${-(axlelength/2) - 0.05}" axle="1" position="-1" upper="0.393" lower="-0.785" />
-        <xacro:car_back_wheel leftright="left" lr="${(axlelength/2) + 0.05}" axle="-1"  upper="3.14" lower="3.14" />
-        <xacro:car_back_wheel leftright="right" lr="${-(axlelength/2) - 0.05}" axle="-1"  upper="3.14" lower="-3.14" />
+        <xacro:car_back_wheel leftright="left" lr="${(axlelength/2) + 0.05}" axle="-1"  upper="${3.14*1000}" lower="${-3.14*1000}" />
+        <xacro:car_back_wheel leftright="right" lr="${-(axlelength/2) - 0.05}" axle="-1"  upper="${3.14*1000}" lower="${-3.14*1000}" />
         <!--
         -->

Commit message: Using a tf Broadcaster to Move the Car in RViz

File: src/car_model/urdf/carModel.urdf (robot description, URDF)
Before this commit: robot car_model, 7 links, 6 joints
Links:
- added link world
Joints:
- added joint world_to_base: type continuous, parent world, child base_link

Commit message: Working on Gazebo Model

File: src/car_model/urdf/carModel.urdf (robot description, URDF)
Before this commit: robot car_model, 8 links, 7 joints
Links:
- removed link world
- added link base_footprint, mass 0.0001; visual box size=0.001 0.001 0.001
Joints:
- removed joint world_to_base
- added joint base_footprint_joint: type fixed, parent base_footprint, child base_link, origin xyz=0 0 0
- joint back_axle_to_base: parent base_link -> base_footprint
- joint back_left_wheel_to_back_axle: parent base_link -> base_footprint
- joint back_right_wheel_to_back_axle: parent base_link -> base_footprint
- joint front_axle_to_base: parent base_link -> base_footprint
- joint front_left_wheel_to_front_axle: parent base_link -> base_footprint
- joint front_right_wheel_to_front_axle: parent base_link -> base_footprint

File: src/car_model/urdf/carModel.xacro (robot description, xacro)
@@ -17,4 +17,5 @@
         <xacro:property name="baseheight" value="${wheelradius}" />
         <xacro:property name="axlelength" value="0.4" />
+        <xacro:property name="update_rate" value="1" />
         <xacro:macro name="default_inertial" params="mass">
           <inertial>
@@ -23,8 +24,22 @@
           </inertial>
         </xacro:macro>
-        <xacro:macro name="global_joint" params="child">
-                <joint name="world_joint_to_${child}" type="fixed">
-                        <parent link="world" />
-                        <child link="${child}" />
+        <xacro:macro name="world_link">
+                <link name="base_footprint">
+                        <visual>
+                                <geometry>
+                                <box size="0.001 0.001 0.001"/>
+                                </geometry>
+                                <origin rpy="0 0 0" xyz="0 0 0"/>
+                        </visual>
+                        <xacro:default_inertial mass="0.0001"/>
+                </link>
+                <gazebo reference="base_footprint">
+                        <material>Gazebo/Green</material>
+                        <turnGravityOff>false</turnGravityOff>
+                </gazebo>
+                <joint name="base_footprint_joint" type="fixed">
+                        <origin xyz="0 0 0" />
+                        <parent link="base_footprint" />
+                        <child link="base_link" />
                 </joint>
         </xacro:macro>
@@ -46,4 +61,7 @@
                         <xacro:default_inertial mass="5"/>
                 </link>
+                <gazebo reference="base_link">
+                        <material>Gazebo/Black</material>
+                </gazebo>
         </xacro:macro>
         <xacro:macro name="car_axle" params="frontback position upper lower">
@@ -65,11 +83,11 @@
                         <axis xyz="1 0 0" />
                         <limit lower="${lower}" upper="${upper}" effort="1000.0" velocity="1.0"/>
-                        <parent link="base_link" />
+                        <parent link="base_footprint" />
                         <child link="${frontback}_axle" />
                         <origin rpy="0 -1.57 0" xyz="0 ${position * 0.3} ${baseheight}" />
                 </joint>
-                <!--
-                <xacro:global_joint child="${frontback}_axle"/>
-        -->
+                <gazebo reference="${frontback}_axle">
+                        <material>Gazebo/Grey</material>
+                </gazebo>
         </xacro:macro>
         <xacro:macro name="car_front_wheel" params="leftright lr axle position upper lower">
@@ -91,11 +109,11 @@
                         <axis xyz="1 0 0" />
                         <limit lower="${lower}" upper="${upper}" effort="1000.0" velocity="1.0"/>
-                        <parent link="base_link" />
+                        <parent link="base_footprint" />
                         <child link="front_${leftright}_wheel" />
                         <origin rpy="0 -1.57 0" xyz="${-lr} 0.3 ${baseheight}" />
                 </joint>
-                <!--
-                <xacro:global_joint child="front_${leftright}_wheel" />
-                -->
+                <gazebo reference="front_${leftright}_wheel">
+                        <material>Gazebo/White</material>
+                </gazebo>
         </xacro:macro>
         <xacro:macro name="car_back_wheel" params="leftright axle lr upper lower">
@@ -117,12 +135,13 @@
                         <axis xyz="0 0 1" />
                         <limit lower="${lower}" upper="${upper}" effort="1000.0" velocity="1.0"/>
-                        <parent link="base_link" />
+                        <parent link="base_footprint" />
                         <child link="back_${leftright}_wheel" />
                         <origin rpy="0 -1.57 0" xyz="${-lr} -0.3 ${baseheight}" />
                 </joint>
-                <!--
-                <xacro:global_joint child="back_${leftright}_wheel"/>
-        -->
+                <gazebo reference="back_${leftright}_wheel">
+                        <material>Gazebo/White</material>
+                </gazebo>
         </xacro:macro>
+        <xacro:world_link />
         <xacro:car_base />
         <xacro:car_axle frontback="front" position="1" upper="0.785" lower="-0.785" />
@@ -134,3 +153,23 @@
         <!--
         -->
+        <gazebo>
+                <plugin name="differential_drive_controller" filename="libgazebo_ros_diff_drive.so">
+                        <alwaysOn>true</alwaysOn>
+                        <legacyMode>false</legacyMode>
+                        <updateRate>${update_rate}</updateRate>
+                        <leftJoint>front_left_wheel_to_front_axle</leftJoint>
+                        <rightJoint>front_right_wheel_to_front_axle</rightJoint>
+                        <wheelSeparation>${axlelength}</wheelSeparation>
+                        <wheelDiameter>${wheelradius * 2}</wheelDiameter>
+                        <torque>20</torque>
+                        <commandTopic>cmd_vel</commandTopic>
+                        <odometryTopic>odom</odometryTopic>
+                        <odometryFrame>odom</odometryFrame>
+                        <robotBaseFrame>base_footprint</robotBaseFrame>
+                        <publishWheelTF>true</publishWheelTF>
+                        <publishTF>100</publishTF>
+                        <publishWheelJointState>true</publishWheelJointState>
+                        <wheelAcceleration>2</wheelAcceleration>
+                </plugin>
+        </gazebo>
 </robot>

Commit message: Working on Odometry

File: src/car_model/urdf/carModel.urdf (robot description, URDF)
Before this commit: robot car_model, 8 links, 7 joints
Links:
- link base_footprint: geometry collision box size=0.001 0.001 0.001; visual box size=0.001 0.001 0.001
Joints:
- joint back_axle_to_base: axis 1 0 0 -> 0 0 1; mimic (none) -> joint=base_footprint_joint multiplier=1; type revolute -> continuous
- joint base_footprint_joint: axis (none) -> 0 0 1; type fixed -> continuous
- joint front_axle_to_base: axis 1 0 0 -> 0 0 1; mimic (none) -> joint=base_footprint_joint multiplier=1; type revolute -> continuous

File: src/car_model/urdf/carModel.xacro (robot description, xacro)
@@ -32,4 +32,10 @@
                                 <origin rpy="0 0 0" xyz="0 0 0"/>
                         </visual>
+                        <collision>
+                                <geometry>
+                                <box size="0.001 0.001 0.001"/>
+                                </geometry>
+                                <origin rpy="0 0 0" xyz="0 0 0"/>
+                        </collision>
                         <xacro:default_inertial mass="0.0001"/>
                 </link>
@@ -38,9 +44,4 @@
                         <turnGravityOff>false</turnGravityOff>
                 </gazebo>
-                <joint name="base_footprint_joint" type="fixed">
-                        <origin xyz="0 0 0" />
-                        <parent link="base_footprint" />
-                        <child link="base_link" />
-                </joint>
         </xacro:macro>
         <xacro:macro name="car_base">
@@ -61,4 +62,10 @@
                         <xacro:default_inertial mass="5"/>
                 </link>
+                <joint name="base_footprint_joint" type="fixed">
+                        <axis xyz="0 0 1" />
+                        <origin xyz="0 0 0" />
+                        <parent link="base_footprint" />
+                        <child link="base_link" />
+                </joint>
                 <gazebo reference="base_link">
                         <material>Gazebo/Black</material>
@@ -66,29 +73,30 @@
         </xacro:macro>
         <xacro:macro name="car_axle" params="frontback position upper lower">
-                <link name="${frontback}_axle">
-                        <visual>
-                                <geometry>
-                                        <cylinder radius="${baselength/8}" length="${axlelength}" />
-                                </geometry>
-                                <material name="gray" />
-                        </visual>
-                        <collision>
-                                <geometry>
-                                        <cylinder radius="${baselength/8}" length="${axlelength}" />
-                                </geometry>
-                        </collision>
-                        <xacro:default_inertial mass="3"/>
-                </link>
-                <joint name="${frontback}_axle_to_base" type="revolute">
-                        <axis xyz="1 0 0" />
-                        <limit lower="${lower}" upper="${upper}" effort="1000.0" velocity="1.0"/>
-                        <parent link="base_footprint" />
-                        <child link="${frontback}_axle" />
-                        <origin rpy="0 -1.57 0" xyz="0 ${position * 0.3} ${baseheight}" />
-                </joint>
-                <gazebo reference="${frontback}_axle">
-                        <material>Gazebo/Grey</material>
-                </gazebo>
-        </xacro:macro>
+                       <link name="${frontback}_axle">
+                               <visual>
+                                       <geometry>
+                                               <cylinder radius="${baselength/8}" length="${axlelength}" />
+                                       </geometry>
+                                       <material name="gray" />
+                               </visual>
+                               <collision>
+                                       <geometry>
+                                               <cylinder radius="${baselength/8}" length="${axlelength}" />
+                                       </geometry>
+                               </collision>
+                               <xacro:default_inertial mass="3"/>
+                       </link>
+                       <joint name="${frontback}_axle_to_base" type="fixed">
+                               <axis xyz="1 0 0" />
+                               <limit lower="${lower}" upper="${upper}" effort="1000.0" velocity="1.0"/>
+                               <mimic joint="base_footprint_joint" multiplier="1"/>
+                               <parent link="base_footprint" />
+                               <child link="${frontback}_axle" />
+                               <origin rpy="0 -1.57 0" xyz="0 ${position * 0.3} ${baseheight}" />
+                       </joint>
+                       <gazebo reference="${frontback}_axle">
+                               <material>Gazebo/Grey</material>
+                       </gazebo>
+               </xacro:macro>
         <xacro:macro name="car_front_wheel" params="leftright lr axle position upper lower">
                 <link name="front_${leftright}_wheel">
@@ -152,13 +160,10 @@
         <xacro:car_back_wheel leftright="right" lr="${-(axlelength/2) - 0.05}" axle="-1"  upper="${3.14*1000}" lower="${-3.14*1000}" />
         <!--
-        -->
+-->
         <gazebo>
                 <plugin name="differential_drive_controller" filename="libgazebo_ros_diff_drive.so">
                         <alwaysOn>true</alwaysOn>
                         <commandTopic>cmd_vel</commandTopic>
-                        <!--
                         <leftJoint>front_right_wheel_to_front_axle</leftJoint>
-                        -->
-                        <leftJoint>back_right_wheel_to_back_axle</leftJoint>
                         <legacyMode>false</legacyMode>
                         <odometryFrame>odom</odometryFrame>
@@ -168,8 +173,5 @@
                         <publishWheelJointState>false</publishWheelJointState>
                         <publishWheelTF>true</publishWheelTF>
-                        <!--
                         <rightJoint>front_left_wheel_to_front_axle</rightJoint>
-                        -->
-                        <rightJoint>back_left_wheel_to_back_axle</rightJoint>
                         <robotBaseFrame>base_footprint</robotBaseFrame>
                         <rosDebugLevel>na</rosDebugLevel>
@@ -181,3 +183,9 @@
                 </plugin>
         </gazebo>
+        <!--
+        <leftJoint>front_right_wheel_to_front_axle</leftJoint>
+        <rightJoint>front_left_wheel_to_front_axle</rightJoint>
+        <leftJoint>back_right_wheel_to_back_axle</leftJoint>
+        <rightJoint>back_left_wheel_to_back_axle</rightJoint>
+        -->
 </robot>

Commit message: Added Simple Camera to Car Model
run Gazebo and RViz at the same time; camera angle is incorrect.

File: src/car_model/urdf/carModel.urdf (robot description, URDF)
Before this commit: robot car_model, 8 links, 7 joints
Links:
- added link camera, mass 1e-05; collision box size=0.1 0.1 0.1; visual box size=0.1 0.1 0.1
Joints:
- added joint camera_joint: type fixed, parent base_footprint, child camera, origin xyz=0 0.3125 0.1875 rpy=0 0 0, axis 0 0 1
- joint back_axle_to_base: axis 0 0 1 -> 1 0 0; type continuous -> fixed
- joint base_footprint_joint: type continuous -> fixed
- joint front_axle_to_base: axis 0 0 1 -> 1 0 0; type continuous -> fixed

File: src/car_model/urdf/carModel.xacro (robot description, xacro)
@@ -151,6 +151,70 @@
                 </gazebo>
         </xacro:macro>
+        <xacro:macro name="camera_link" params="height width">
+                <link name="camera">
+                        <visual>
+                                <geometry>
+                                        <box size="0.1 0.1 0.1"/>
+                                </geometry>
+                                <material name="blue"/>
+                        </visual>
+                        <collision>
+                                <geometry>
+                                        <box size="0.1 0.1 0.1"/>
+                                </geometry>
+                        </collision>
+                        <xacro:default_inertial mass="1e-5"/>
+                </link>
+                <joint name="camera_joint" type="fixed">
+                        <axis xyz="0 0 1" />
+                        <origin xyz="0 ${(baselength/2)+(baselength/4)} ${baseheight+(baselength/8)}" rpy="1.57 0 0"/>
+                        <parent link="base_footprint"/>
+                        <child link="camera"/>
+                </joint>
+                <gazebo reference="camera">
+                        <material>Gazebo/Blue</material>
+                        <!--from http://gazebosim.org/tutorials?tut=ros_gzplugins-->
+                        <sensor type="camera" name="car_model_camera">
+                                <update_rate>33.3</update_rate>
+                                <camera name="camera">
+                                        <horizontal_fov>1.3962634</horizontal_fov>
+                                        <image>
+                                                <width>${width}</width>
+                                                <height>${height}</height>
+                                                <format>R8G8B8</format>
+                                        </image>
+                                        <clip>
+                                                <near>0.02</near>
+                                                <far>300</far>
+                                        </clip>
+                                        <noise>
+                                                <type>gaussian</type>
+                                                <!-- Noise is sampled independently per pixel on each frame.
+                                                That pixel's noise value is added to each of its color
+                                                channels, which at that point lie in the range [0,1]. -->
+                                                <mean>0.0</mean>
+                                                <stddev>0.007</stddev>
+                                        </noise>
+                                </camera>
+                                <plugin name="camera_controller" filename="libgazebo_ros_camera.so">
+                                        <alwaysOn>true</alwaysOn>
+                                        <updateRate>0.0</updateRate>
+                                        <cameraName>car_model_camera</cameraName>
+                                        <imageTopicName>image_raw</imageTopicName>
+                                        <cameraInfoTopicName>camera_info</cameraInfoTopicName>
+                                        <frameName>odom</frameName>
+                                        <hackBaseline>0.07</hackBaseline>
+                                        <distortionK1>0.0</distortionK1>
+                                        <distortionK2>0.0</distortionK2>
+                                        <distortionK3>0.0</distortionK3>
+                                        <distortionT1>0.0</distortionT1>
+                                        <distortionT2>0.0</distortionT2>
+                                </plugin>
+                        </sensor>
+                </gazebo>
+        </xacro:macro>
         <xacro:world_link />
         <xacro:car_base />
+        <xacro:camera_link height="480" width="640" />
         <xacro:car_axle frontback="front" position="1" upper="0.785" lower="-0.785" />
         <xacro:car_axle frontback="back" position="-1" upper="0.785" lower="-0.785" />
