Commit message: Camera Now Points Ahead of Car

File: src/car_model/urdf/carModel.urdf (robot description, URDF)
Before this commit: robot car_model, 9 links, 8 joints
Links:
- link back_axle: mass 3 -> 10
- link base_link: mass 5 -> 15
- link front_axle: mass 3 -> 10
Joints:
- joint camera_joint: axis 0 0 1 -> (none); origin xyz=0 0.3125 0.1875 rpy=0 0 0 -> xyz=0 0.375 0.1875 rpy=-1.57 -1.57 1.57; type fixed -> continuous

File: src/car_model/urdf/carModel.xacro (robot description, xacro)
@@ -42,5 +42,4 @@
                 <gazebo reference="base_footprint">
                         <material>Gazebo/Green</material>
-                        <turnGravityOff>false</turnGravityOff>
                 </gazebo>
         </xacro:macro>
@@ -60,5 +59,5 @@
                                 <origin rpy="0 0 0" xyz="0 0 ${baseheight}" />
                         </collision>
-                        <xacro:default_inertial mass="5"/>
+                        <xacro:default_inertial mass="15"/>
                 </link>
                 <joint name="base_footprint_joint" type="fixed">
@@ -85,5 +84,5 @@
                                        </geometry>
                                </collision>
-                               <xacro:default_inertial mass="3"/>
+                               <xacro:default_inertial mass="10"/>
                        </link>
                        <joint name="${frontback}_axle_to_base" type="fixed">
@@ -121,5 +120,27 @@
                         <origin rpy="0 -1.57 0" xyz="${-lr} 0.3 ${baseheight}" />
                 </joint>
+                <transmission name="front_${leftright}_trans">
+                        <type>transmission_interface/SimpleTransmission</type>
+                        <actuator name="front_${leftright}_motor">
+                                <mechanicalReduction>1</mechanicalReduction>
+                        </actuator>
+                        <joint name="front_${leftright}_wheel_to_front_axle">
+                                <hardwareInterface>hardware_interface/PositionJointInterface</hardwareInterface>
+                        </joint>
+                </transmission>
+                <transmission name="front_${leftright}_vel_trans">
+                        <type>transmission_interface/SimpleTransmission</type>
+                        <actuator name="front_${leftright}_vel_motor">
+                                <mechanicalReduction>1</mechanicalReduction>
+                        </actuator>
+                        <joint name="front_${leftright}_wheel_to_front_axle">
+                                <hardwareInterface>hardware_interface/VelocityJointInterface</hardwareInterface>
+                        </joint>
+                </transmission>
                 <gazebo reference="front_${leftright}_wheel">
+                        <mu1 value="200.0"/>
+                        <mu2 value="100.0"/>
+                        <kp value="10000000.0" />
+                        <kd value="1.0" />
                         <material>Gazebo/White</material>
                 </gazebo>
@@ -147,5 +168,27 @@
                         <origin rpy="0 -1.57 0" xyz="${-lr} -0.3 ${baseheight}" />
                 </joint>
+                <transmission name="back_${leftright}_trans">
+                        <type>transmission_interface/SimpleTransmission</type>
+                        <actuator name="back_${leftright}_motor">
+                                <mechanicalReduction>1</mechanicalReduction>
+                        </actuator>
+                        <joint name="back_${leftright}_wheel_to_back_axle">
+                                <hardwareInterface>hardware_interface/PositionJointInterface</hardwareInterface>
+                        </joint>
+                </transmission>
+                <transmission name="back_${leftright}_vel_trans">
+                        <type>transmission_interface/SimpleTransmission</type>
+                        <actuator name="back_${leftright}_vel_motor">
+                                <mechanicalReduction>1</mechanicalReduction>
+                        </actuator>
+                        <joint name="back_${leftright}_wheel_to_back_axle">
+                                <hardwareInterface>hardware_interface/VelocityJointInterface</hardwareInterface>
+                        </joint>
+                </transmission>
                 <gazebo reference="back_${leftright}_wheel">
+                        <mu1 value="200.0"/>
+                        <mu2 value="100.0"/>
+                        <kp value="10000000.0" />
+                        <kd value="1.0" />
                         <material>Gazebo/White</material>
                 </gazebo>
@@ -157,5 +200,5 @@
                                         <box size="0.1 0.1 0.1"/>
                                 </geometry>
-                                <material name="blue"/>
+                                <material name="black"/>
                         </visual>
                         <collision>
@@ -168,11 +211,10 @@
                 <joint name="camera_joint" type="fixed">
                         <axis xyz="0 0 1" />
-                        <origin xyz="0 ${(baselength/2)+(baselength/4)} ${baseheight+(baselength/8)}" rpy="1.57 0 0"/>
+                        <origin xyz="0 ${(baselength/2)+(baselength/4)} ${baseheight}" rpy="0 0 1.57"/>
                         <parent link="base_footprint"/>
                         <child link="camera"/>
                 </joint>
                 <gazebo reference="camera">
-                        <material>Gazebo/Blue</material>
-                        <!--from http://gazebosim.org/tutorials?tut=ros_gzplugins-->
+                        <material>Gazebo/Black</material>
                         <sensor type="camera" name="car_model_camera">
                                 <update_rate>33.3</update_rate>
@@ -190,7 +232,4 @@
                                         <noise>
                                                 <type>gaussian</type>
-                                                <!-- Noise is sampled independently per pixel on each frame.
-                                                That pixel's noise value is added to each of its color
-                                                channels, which at that point lie in the range [0,1]. -->
                                                 <mean>0.0</mean>
                                                 <stddev>0.007</stddev>
@@ -226,8 +265,13 @@
 -->
         <gazebo>
+<!--
+                <plugin name="gazebo_ros_control" filename="libgazebo_ros_control.so">
+                        <robotNamespace>/</robotNamespace>
+                </plugin>
+-->
                 <plugin name="differential_drive_controller" filename="libgazebo_ros_diff_drive.so">
                         <alwaysOn>true</alwaysOn>
                         <commandTopic>cmd_vel</commandTopic>
-                        <leftJoint>front_left_wheel_to_front_axle</leftJoint>
+                        <leftJoint>[front_left_wheel_to_front_axle, back_left_wheel_to_back_axle]</leftJoint>
                         <legacyMode>false</legacyMode>
                         <odometryFrame>odom</odometryFrame>
@@ -236,5 +280,5 @@
                         <publishWheelJointState>false</publishWheelJointState>
                         <publishWheelTF>true</publishWheelTF>
-                        <rightJoint>front_right_wheel_to_front_axle</rightJoint>
+                        <rightJoint>[front_right_wheel_to_front_axle, back_right_wheel_to_back_axle]</rightJoint>
                         <robotBaseFrame>base_link</robotBaseFrame>
                         <robotNamespace>robot::base_footprint</robotNamespace>
