Commit message: Updated URDF, RViz, and Launch Files

File: src/car_model/urdf/gazeboCar.xacro (robot description, xacro)
@@ -17,9 +17,16 @@
         <xacro:property name="baseheight" value="${wheelradius}" />
         <xacro:property name="axlelength" value="0.4" />
-        <xacro:property name="update_rate" value="1.0" />
+        <xacro:property name="update_rate" value="5.0" />
         <xacro:property name="base_mass" value="1e-1" />
         <xacro:property name="axle_mass" value="${0.5*1e-1}" />
         <xacro:property name="wheel_mass" value="1e+0" />
         <xacro:property name="camera_mass" value="1e-2" />
+        <xacro:macro name="gazebo_wheel_elements" >
+                <mu1 value="300.0"/>
+                <mu2 value="100.0"/>
+                <kp value="100000.0" />
+                <kd value="1.0" />
+                <material>Gazebo/White</material>
+        </xacro:macro>
         <xacro:macro name="default_inertial" params="mass">
                 <inertial>
@@ -43,4 +50,7 @@
                         <xacro:default_inertial mass="${base_mass/100}"/>
                 </link>
+                <gazebo reference="base_footprint">
+                        <material>Gazebo/Green</material>
+                </gazebo>
         </xacro:macro>
         <xacro:macro name="car_base">
@@ -65,4 +75,7 @@
                         <origin rpy="0 0 0" xyz="0 0 ${baseheight}" />
                 </joint>
+                <gazebo reference="base_link">
+                        <material>Gazebo/Black</material>
+                </gazebo>
         </xacro:macro>
         <xacro:macro name="car_axle" params="frontback position upper lower">
@@ -89,7 +102,10 @@
                        <origin rpy="0 -1.57 0" xyz="0 ${position * 0.3} ${baseheight}" />
                </joint>
+               <gazebo reference="${frontback}_axle">
+                       <material>Gazebo/Grey</material>
+               </gazebo>
        </xacro:macro>
-        <xacro:macro name="car_front_wheel" params="leftright lr axle position upper lower">
-                <link name="front_${leftright}_wheel">
+        <xacro:macro name="car_wheel" params="frontback leftright fb lr">
+                <link name="${frontback}_${leftright}_wheel">
                         <visual>
                                 <geometry>
@@ -105,33 +121,13 @@
                         <xacro:default_inertial mass="${wheel_mass}"/>
                 </link>
-                <joint name="front_${leftright}_wheel_to_front_axle" type="revolute">
-                        <axis xyz="1 0 0" />
-                        <limit lower="${lower}" upper="${upper}" effort="1000.0" velocity="1.0"/>
-                        <parent link="base_footprint" />
-                        <child link="front_${leftright}_wheel" />
-                        <origin rpy="0 -1.57 0" xyz="${-lr} 0.3 ${baseheight}" />
-                </joint>
-        </xacro:macro>
-        <xacro:macro name="car_back_wheel" params="leftright axle lr upper lower">
-                <link name="back_${leftright}_wheel">
-                        <visual>
-                                <geometry>
-                                        <cylinder radius="${wheelradius}" length="${wheelradius}" />
-                                </geometry>
-                                <material name="white" />
-                        </visual>
-                        <collision>
-                                <geometry>
-                                        <cylinder radius="${wheelradius}" length="${wheelradius}" />
-                                </geometry>
-                        </collision>
-                        <xacro:default_inertial mass="${wheel_mass}"/>
-                </link>
-                <joint name="back_${leftright}_wheel_to_back_axle" type="continuous">
+                <joint name="${frontback}_${leftright}_wheel_to_${frontback}_axle" type="continuous">
                         <axis xyz="0 0 1" />
                         <parent link="base_footprint" />
-                        <child link="back_${leftright}_wheel" />
-                        <origin rpy="0 -1.57 0" xyz="${-lr} -0.3 ${baseheight}" />
+                        <child link="${frontback}_${leftright}_wheel" />
+                        <origin rpy="0 -1.57 0" xyz="${-lr} ${fb} ${baseheight}" />
                 </joint>
+                <gazebo reference="${frontback}_${leftright}_wheel">
+                        <xacro:gazebo_wheel_elements />
+                </gazebo>
         </xacro:macro>
         <xacro:macro name="camera_link" params="height width">
@@ -156,4 +152,41 @@
                         <child link="camera"/>
                 </joint>
+                <gazebo reference="camera">
+                        <material>Gazebo/Black</material>
+                        <sensor type="camera" name="car_model_camera">
+                                <update_rate>33.3</update_rate>
+                                <camera name="camera">
+                                        <horizontal_fov>1.3962634</horizontal_fov>
+                                        <image>
+                                                <width>${width}</width>
+                                                <height>${height}</height>
+                                                <format>R8G8B8</format>
+                                        </image>
+                                        <clip>
+                                                <near>0.02</near>
+                                                <far>300</far>
+                                        </clip>
+                                        <noise>
+                                                <type>gaussian</type>
+                                                <mean>0.0</mean>
+                                                <stddev>0.007</stddev>
+                                        </noise>
+                                </camera>
+                                <plugin name="camera_controller" filename="libgazebo_ros_camera.so">
+                                        <alwaysOn>true</alwaysOn>
+                                        <updateRate>0.00</updateRate>
+                                        <cameraName>car_model_camera</cameraName>
+                                        <imageTopicName>image_raw</imageTopicName>
+                                        <cameraInfoTopicName>camera_info</cameraInfoTopicName>
+                                        <frameName>odom</frameName>
+                                        <hackBaseline>0.07</hackBaseline>
+                                        <distortionK1>0.0</distortionK1>
+                                        <distortionK2>0.0</distortionK2>
+                                        <distortionK3>0.0</distortionK3>
+                                        <distortionT1>0.0</distortionT1>
+                                        <distortionT2>0.0</distortionT2>
+                                </plugin>
+                        </sensor>
+                </gazebo>
         </xacro:macro>
         <xacro:world_link />
@@ -162,11 +195,30 @@
         <xacro:car_axle frontback="front" position="1" upper="0.785" lower="-0.785" />
         <xacro:car_axle frontback="back" position="-1" upper="0.785" lower="-0.785" />
-        <xacro:car_front_wheel leftright="left" lr="${(axlelength/2) + 0.05}" axle="1"
-                position="1" upper="0.785" lower="-0.393" />
-        <xacro:car_front_wheel leftright="right" lr="${-(axlelength/2) - 0.05}" axle="1"
-                position="-1" upper="0.393" lower="-0.785" />
-        <xacro:car_back_wheel leftright="left" lr="${(axlelength/2) + 0.05}" axle="-1"
-                upper="${3.14*1000}" lower="${-3.14*1000}" />
-        <xacro:car_back_wheel leftright="right" lr="${-(axlelength/2) - 0.05}" axle="-1"
-                upper="${3.14*1000}" lower="${-3.14*1000}" />
+        <xacro:car_wheel frontback="front" leftright="left" fb="0.3" lr="${(axlelength/2) + 0.05}" />
+        <xacro:car_wheel frontback="front" leftright="right" fb="0.3" lr="${-(axlelength/2) - 0.05}" />
+        <xacro:car_wheel frontback="back" leftright="left" fb="-0.3" lr="${(axlelength/2) + 0.05}" />
+        <xacro:car_wheel frontback="back" leftright="right" fb="-0.3" lr="${-(axlelength/2) - 0.05}" />
+        <gazebo>
+                <plugin name="skid_steer_drive_controller" filename="libgazebo_ros_skid_steer_drive.so">
+                        <broadcastTF>true</broadcastTF>
+                        <commandTopic>cmd_vel</commandTopic>
+                        <covariance_x>0.000100</covariance_x>
+                        <covariance_y>0.000100</covariance_y>
+                        <covariance_yaw>0.010000</covariance_yaw>
+                        <leftFrontJoint>front_left_wheel_to_front_axle</leftFrontJoint>
+                        <leftRearJoint>back_left_wheel_to_back_axle</leftRearJoint>
+                        <odometryFrame>odom</odometryFrame>
+                        <odometryTopic>odom</odometryTopic>
+                        <rightFrontJoint>front_right_wheel_to_front_axle</rightFrontJoint>
+                        <rightRearJoint>back_right_wheel_to_back_axle</rightRearJoint>
+                        <robotBaseFrame>base_footprint</robotBaseFrame>
+                        <robotNamespace>/</robotNamespace>
+                        <topicName>cmd_vel</topicName>
+                        <torque>18</torque>
+                        <updateRate>100.0</updateRate>
+                        <wheelDiameter>${wheelradius * 2}</wheelDiameter>
+                        <wheelSeparation>${axlelength}</wheelSeparation>
+                </plugin>
+                <plugin name="gazebo_ros_control" filename="libgazebo_ros_control.so" />
+        </gazebo>
 </robot>
