Commit message: Updating TF Angle Calculation

File: src/car_model/urdf/carModel.xacro (robot description, xacro)
@@ -17,5 +17,5 @@
         <xacro:property name="baseheight" value="${wheelradius}" />
         <xacro:property name="axlelength" value="0.4" />
-        <xacro:property name="update_rate" value="1" />
+        <xacro:property name="update_rate" value="0.5" />
         <xacro:macro name="default_inertial" params="mass">
           <inertial>
@@ -156,19 +156,27 @@
                 <plugin name="differential_drive_controller" filename="libgazebo_ros_diff_drive.so">
                         <alwaysOn>true</alwaysOn>
+                        <commandTopic>cmd_vel</commandTopic>
+                        <!--
+                        <leftJoint>front_right_wheel_to_front_axle</leftJoint>
+                        -->
+                        <leftJoint>back_right_wheel_to_back_axle</leftJoint>
                         <legacyMode>false</legacyMode>
+                        <odometryFrame>odom</odometryFrame>
+                        <odometrySource>1</odometrySource>
+                        <odometryTopic>odom</odometryTopic>
+                        <publishTf>10</publishTf>
+                        <publishWheelJointState>false</publishWheelJointState>
+                        <publishWheelTF>true</publishWheelTF>
+                        <!--
+                        <rightJoint>front_left_wheel_to_front_axle</rightJoint>
+                        -->
+                        <rightJoint>back_left_wheel_to_back_axle</rightJoint>
+                        <robotBaseFrame>base_footprint</robotBaseFrame>
+                        <rosDebugLevel>na</rosDebugLevel>
+                        <wheelTorque>5</wheelTorque>
                         <updateRate>${update_rate}</updateRate>
-                        <leftJoint>front_left_wheel_to_front_axle</leftJoint>
-                        <rightJoint>front_right_wheel_to_front_axle</rightJoint>
+                        <wheelAcceleration>2</wheelAcceleration>
+                        <wheelDiameter>${wheelradius * 2}</wheelDiameter>
                         <wheelSeparation>${axlelength}</wheelSeparation>
-                        <wheelDiameter>${wheelradius * 2}</wheelDiameter>
-                        <torque>20</torque>
-                        <commandTopic>cmd_vel</commandTopic>
-                        <odometryTopic>odom</odometryTopic>
-                        <odometryFrame>odom</odometryFrame>
-                        <robotBaseFrame>base_footprint</robotBaseFrame>
-                        <publishWheelTF>true</publishWheelTF>
-                        <publishTF>100</publishTF>
-                        <publishWheelJointState>true</publishWheelJointState>
-                        <wheelAcceleration>2</wheelAcceleration>
                 </plugin>
         </gazebo>

Commit message: Working on Odometry and Gazebo

File: src/car_model/urdf/carModel.xacro (robot description, xacro)
@@ -17,5 +17,5 @@
         <xacro:property name="baseheight" value="${wheelradius}" />
         <xacro:property name="axlelength" value="0.4" />
-        <xacro:property name="update_rate" value="0.5" />
+        <xacro:property name="update_rate" value="0.1" />
         <xacro:macro name="default_inertial" params="mass">
           <inertial>

Commit message: Finished Video-to-Image Converter; Started Stream Converter

File: src/car_model/urdf/carModel.xacro (robot description, xacro)
@@ -19,8 +19,8 @@
         <xacro:property name="update_rate" value="0.1" />
         <xacro:macro name="default_inertial" params="mass">
-          <inertial>
-            <mass value="${mass}" />
-            <inertia ixx="1.0" ixy="0.0" ixz="0.0" iyy="1.0" iyz="0.0" izz="1.0" />
-          </inertial>
+                <inertial>
+                        <mass value="${mass}" />
+                        <inertia ixx="1.0" ixy="0.0" ixz="0.0" iyy="1.0" iyz="0.0" izz="1.0" />
+                </inertial>
         </xacro:macro>
         <xacro:macro name="world_link">
@@ -72,30 +72,30 @@
         </xacro:macro>
         <xacro:macro name="car_axle" params="frontback position upper lower">
-                       <link name="${frontback}_axle">
-                               <visual>
-                                       <geometry>
-                                               <cylinder radius="${baselength/8}" length="${axlelength}" />
-                                       </geometry>
-                                       <material name="gray" />
-                               </visual>
-                               <collision>
-                                       <geometry>
-                                               <cylinder radius="${baselength/8}" length="${axlelength}" />
-                                       </geometry>
-                               </collision>
-                               <xacro:default_inertial mass="10"/>
-                       </link>
-                       <joint name="${frontback}_axle_to_base" type="fixed">
-                               <axis xyz="1 0 0" />
-                               <limit lower="${lower}" upper="${upper}" effort="1000.0" velocity="1.0"/>
-                               <mimic joint="base_footprint_joint" multiplier="1"/>
-                               <parent link="base_footprint" />
-                               <child link="${frontback}_axle" />
-                               <origin rpy="0 -1.57 0" xyz="0 ${position * 0.3} ${baseheight}" />
-                       </joint>
-                       <gazebo reference="${frontback}_axle">
-                               <material>Gazebo/Grey</material>
-                       </gazebo>
-               </xacro:macro>
+               <link name="${frontback}_axle">
+                       <visual>
+                               <geometry>
+                                       <cylinder radius="${baselength/8}" length="${axlelength}" />
+                               </geometry>
+                               <material name="gray" />
+                       </visual>
+                       <collision>
+                               <geometry>
+                                       <cylinder radius="${baselength/8}" length="${axlelength}" />
+                               </geometry>
+                       </collision>
+                       <xacro:default_inertial mass="10"/>
+               </link>
+               <joint name="${frontback}_axle_to_base" type="fixed">
+                       <axis xyz="1 0 0" />
+                       <limit lower="${lower}" upper="${upper}" effort="1000.0" velocity="1.0"/>
+                       <mimic joint="base_footprint_joint" multiplier="1"/>
+                       <parent link="base_footprint" />
+                       <child link="${frontback}_axle" />
+                       <origin rpy="0 -1.57 0" xyz="0 ${position * 0.3} ${baseheight}" />
+               </joint>
+               <gazebo reference="${frontback}_axle">
+                       <material>Gazebo/Grey</material>
+               </gazebo>
+       </xacro:macro>
         <xacro:macro name="car_front_wheel" params="leftright lr axle position upper lower">
                 <link name="front_${leftright}_wheel">
@@ -258,29 +258,34 @@
         <xacro:car_axle frontback="front" position="1" upper="0.785" lower="-0.785" />
         <xacro:car_axle frontback="back" position="-1" upper="0.785" lower="-0.785" />
-        <xacro:car_front_wheel leftright="left" lr="${(axlelength/2) + 0.05}" axle="1" position="1" upper="0.785" lower="-0.393" />
-        <xacro:car_front_wheel leftright="right" lr="${-(axlelength/2) - 0.05}" axle="1" position="-1" upper="0.393" lower="-0.785" />
-        <xacro:car_back_wheel leftright="left" lr="${(axlelength/2) + 0.05}" axle="-1"  upper="${3.14*1000}" lower="${-3.14*1000}" />
-        <xacro:car_back_wheel leftright="right" lr="${-(axlelength/2) - 0.05}" axle="-1"  upper="${3.14*1000}" lower="${-3.14*1000}" />
+        <xacro:car_front_wheel leftright="left" lr="${(axlelength/2) + 0.05}" axle="1"
+                position="1" upper="0.785" lower="-0.393" />
+        <xacro:car_front_wheel leftright="right" lr="${-(axlelength/2) - 0.05}" axle="1"
+                position="-1" upper="0.393" lower="-0.785" />
+        <xacro:car_back_wheel leftright="left" lr="${(axlelength/2) + 0.05}" axle="-1"
+                upper="${3.14*1000}" lower="${-3.14*1000}" />
+        <xacro:car_back_wheel leftright="right" lr="${-(axlelength/2) - 0.05}" axle="-1"
+                upper="${3.14*1000}" lower="${-3.14*1000}" />
         <!--
 -->
         <gazebo>
-<!--
+                <!--
                 <plugin name="gazebo_ros_control" filename="libgazebo_ros_control.so">
                         <robotNamespace>/</robotNamespace>
                 </plugin>
--->
-                <plugin name="differential_drive_controller" filename="libgazebo_ros_diff_drive.so">
+                -->
+                <plugin name="car_model_diff_drive_controller" filename="libgazebo_ros_diff_drive.so">
                         <alwaysOn>true</alwaysOn>
                         <commandTopic>cmd_vel</commandTopic>
-                        <leftJoint>[front_left_wheel_to_front_axle, back_left_wheel_to_back_axle]</leftJoint>
+                        <leftJoint>front_left_wheel_to_front_axle</leftJoint>
                         <legacyMode>false</legacyMode>
                         <odometryFrame>odom</odometryFrame>
+                        <odometrySource>1</odometrySource>
                         <odometryTopic>odom</odometryTopic>
                         <publishTf>100</publishTf>
                         <publishWheelJointState>false</publishWheelJointState>
                         <publishWheelTF>true</publishWheelTF>
-                        <rightJoint>[front_right_wheel_to_front_axle, back_right_wheel_to_back_axle]</rightJoint>
-                        <robotBaseFrame>base_link</robotBaseFrame>
-                        <robotNamespace>robot::base_footprint</robotNamespace>
+                        <rightJoint>front_right_wheel_to_front_axle</rightJoint>
+                        <robotBaseFrame>base_footprint</robotBaseFrame>
+                        <robotNamespace>robot</robotNamespace>
                         <rosDebugLevel>na</rosDebugLevel>
                         <wheelTorque>5</wheelTorque>

Commit message: Minor Gazebo Changes

File: src/car_model/urdf/carModel.xacro (robot description, xacro)
@@ -17,5 +17,5 @@
         <xacro:property name="baseheight" value="${wheelradius}" />
         <xacro:property name="axlelength" value="0.4" />
-        <xacro:property name="update_rate" value="0.1" />
+        <xacro:property name="update_rate" value="1.0" />
         <xacro:macro name="default_inertial" params="mass">
                 <inertial>
@@ -120,22 +120,4 @@
                         <origin rpy="0 -1.57 0" xyz="${-lr} 0.3 ${baseheight}" />
                 </joint>
-                <transmission name="front_${leftright}_trans">
-                        <type>transmission_interface/SimpleTransmission</type>
-                        <actuator name="front_${leftright}_motor">
-                                <mechanicalReduction>1</mechanicalReduction>
-                        </actuator>
-                        <joint name="front_${leftright}_wheel_to_front_axle">
-                                <hardwareInterface>hardware_interface/PositionJointInterface</hardwareInterface>
-                        </joint>
-                </transmission>
-                <transmission name="front_${leftright}_vel_trans">
-                        <type>transmission_interface/SimpleTransmission</type>
-                        <actuator name="front_${leftright}_vel_motor">
-                                <mechanicalReduction>1</mechanicalReduction>
-                        </actuator>
-                        <joint name="front_${leftright}_wheel_to_front_axle">
-                                <hardwareInterface>hardware_interface/VelocityJointInterface</hardwareInterface>
-                        </joint>
-                </transmission>
                 <gazebo reference="front_${leftright}_wheel">
                         <mu1 value="200.0"/>
@@ -168,22 +150,4 @@
                         <origin rpy="0 -1.57 0" xyz="${-lr} -0.3 ${baseheight}" />
                 </joint>
-                <transmission name="back_${leftright}_trans">
-                        <type>transmission_interface/SimpleTransmission</type>
-                        <actuator name="back_${leftright}_motor">
-                                <mechanicalReduction>1</mechanicalReduction>
-                        </actuator>
-                        <joint name="back_${leftright}_wheel_to_back_axle">
-                                <hardwareInterface>hardware_interface/PositionJointInterface</hardwareInterface>
-                        </joint>
-                </transmission>
-                <transmission name="back_${leftright}_vel_trans">
-                        <type>transmission_interface/SimpleTransmission</type>
-                        <actuator name="back_${leftright}_vel_motor">
-                                <mechanicalReduction>1</mechanicalReduction>
-                        </actuator>
-                        <joint name="back_${leftright}_wheel_to_back_axle">
-                                <hardwareInterface>hardware_interface/VelocityJointInterface</hardwareInterface>
-                        </joint>
-                </transmission>
                 <gazebo reference="back_${leftright}_wheel">
                         <mu1 value="200.0"/>
@@ -238,5 +202,5 @@
                                 <plugin name="camera_controller" filename="libgazebo_ros_camera.so">
                                         <alwaysOn>true</alwaysOn>
-                                        <updateRate>0.0</updateRate>
+                                        <updateRate>0.00</updateRate>
                                         <cameraName>car_model_camera</cameraName>
                                         <imageTopicName>image_raw</imageTopicName>
@@ -270,26 +234,24 @@
         <gazebo>
                 <!--
-                <plugin name="gazebo_ros_control" filename="libgazebo_ros_control.so">
-                        <robotNamespace>/</robotNamespace>
-                </plugin>
-                -->
+        -->
                 <plugin name="car_model_diff_drive_controller" filename="libgazebo_ros_diff_drive.so">
                         <alwaysOn>true</alwaysOn>
                         <commandTopic>cmd_vel</commandTopic>
                         <leftJoint>front_left_wheel_to_front_axle</leftJoint>
-                        <legacyMode>false</legacyMode>
+                        <leftJoint>back_left_wheel_to_back_axle</leftJoint>
+                        <legacyMode>true</legacyMode>
                         <odometryFrame>odom</odometryFrame>
-                        <odometrySource>1</odometrySource>
+                        <odometrySource>odom</odometrySource>
                         <odometryTopic>odom</odometryTopic>
-                        <publishTf>100</publishTf>
+                        <publishTf>false</publishTf>
                         <publishWheelJointState>false</publishWheelJointState>
-                        <publishWheelTF>true</publishWheelTF>
+                        <publishWheelTF>false</publishWheelTF>
                         <rightJoint>front_right_wheel_to_front_axle</rightJoint>
+                        <rightJoint>back_right_wheel_to_back_axle</rightJoint>
                         <robotBaseFrame>base_footprint</robotBaseFrame>
-                        <robotNamespace>robot</robotNamespace>
                         <rosDebugLevel>na</rosDebugLevel>
-                        <wheelTorque>5</wheelTorque>
+                        <wheelTorque>20</wheelTorque>
                         <updateRate>${update_rate}</updateRate>
-                        <wheelAcceleration>2</wheelAcceleration>
+                        <wheelAcceleration>20</wheelAcceleration>
                         <wheelDiameter>${wheelradius * 2}</wheelDiameter>
                         <wheelSeparation>${axlelength}</wheelSeparation>
@@ -297,8 +259,8 @@
         </gazebo>
         <!--
-        <leftJoint>front_right_wheel_to_front_axle</leftJoint>
-        <rightJoint>front_left_wheel_to_front_axle</rightJoint>
-        <leftJoint>back_right_wheel_to_back_axle</leftJoint>
-        <rightJoint>back_left_wheel_to_back_axle</rightJoint>
+        <leftJoint>front_left_wheel_to_front_axle</leftJoint>
+        <rightJoint>front_right_wheel_to_front_axle</rightJoint>
+        <leftJoint>back_left_wheel_to_back_axle</leftJoint>
+        <rightJoint>back_right_wheel_to_back_axle</rightJoint>
         -->
 </robot>
