Commit message: Corrected carModel's Inertia and Collision

File: src/car_model/urdf/carModel.xacro (robot description, xacro)
@@ -18,8 +18,12 @@
         <xacro:property name="axlelength" value="0.4" />
         <xacro:property name="update_rate" value="1.0" />
+        <xacro:property name="base_mass" value="1e-1" />
+        <xacro:property name="axle_mass" value="${0.5*1e-1}" />
+        <xacro:property name="wheel_mass" value="1e+0" />
+        <xacro:property name="camera_mass" value="1e-2" />
         <xacro:macro name="default_inertial" params="mass">
                 <inertial>
                         <mass value="${mass}" />
-                        <inertia ixx="1.0" ixy="0.0" ixz="0.0" iyy="1.0" iyz="0.0" izz="1.0" />
+                        <inertia ixx="${mass*0.01}" ixy="0.0" ixz="0.0" iyy="${mass*0.01}" iyz="0.0" izz="${mass*0.01}" />
                 </inertial>
         </xacro:macro>
@@ -28,5 +32,5 @@
                         <visual>
                                 <geometry>
-                                <box size="0.001 0.001 0.001"/>
+                                        <box size="0.001 0.001 0.001"/>
                                 </geometry>
                                 <origin rpy="0 0 0" xyz="0 0 0"/>
@@ -34,9 +38,8 @@
                         <collision>
                                 <geometry>
-                                <box size="0.001 0.001 0.001"/>
-                                </geometry>
-                                <origin rpy="0 0 0" xyz="0 0 0"/>
-                        </collision>
-                        <xacro:default_inertial mass="0.0001"/>
+                                        <box size="0.001 0.001 0.001"/>
+                                </geometry>
+                        </collision>
+                        <xacro:default_inertial mass="${base_mass/100}"/>
                 </link>
                 <gazebo reference="base_footprint">
@@ -51,5 +54,4 @@
                                 </geometry>
                                 <material name="black" />
-                                <origin rpy="0 0 0" xyz="0 0 ${baseheight}" />
                         </visual>
                         <collision>
@@ -57,13 +59,12 @@
                                         <box size="${baselength/2} ${baselength} ${baselength/8}" />
                                 </geometry>
-                                <origin rpy="0 0 0" xyz="0 0 ${baseheight}" />
-                        </collision>
-                        <xacro:default_inertial mass="15"/>
+                        </collision>
+                        <xacro:default_inertial mass="${base_mass}"/>
                 </link>
                 <joint name="base_footprint_joint" type="fixed">
                         <axis xyz="0 0 1" />
-                        <origin xyz="0 0 0" />
                         <parent link="base_footprint" />
                         <child link="base_link" />
+                        <origin rpy="0 0 0" xyz="0 0 ${baseheight}" />
                 </joint>
                 <gazebo reference="base_link">
@@ -84,5 +85,5 @@
                                </geometry>
                        </collision>
-                       <xacro:default_inertial mass="10"/>
+                       <xacro:default_inertial mass="${axle_mass}"/>
                </link>
                <joint name="${frontback}_axle_to_base" type="fixed">
@@ -111,8 +112,8 @@
                                 </geometry>
                         </collision>
-                        <xacro:default_inertial mass="20"/>
-                </link>
-                <joint name="front_${leftright}_wheel_to_front_axle" type="revolute">
-                        <axis xyz="1 0 0" />
+                        <xacro:default_inertial mass="${wheel_mass}"/>
+                </link>
+                <joint name="front_${leftright}_wheel_to_front_axle" type="continuous">
+                        <axis xyz="0 0 1" />
                         <limit lower="${lower}" upper="${upper}" effort="1000.0" velocity="1.0"/>
                         <parent link="base_footprint" />
@@ -121,7 +122,7 @@
                 </joint>
                 <gazebo reference="front_${leftright}_wheel">
-                        <mu1 value="200.0"/>
-                        <mu2 value="100.0"/>
-                        <kp value="10000000.0" />
+                        <mu1 value="20.0"/>
+                        <mu2 value="10.0"/>
+                        <kp value="10000.0" />
                         <kd value="1.0" />
                         <material>Gazebo/White</material>
@@ -141,7 +142,7 @@
                                 </geometry>
                         </collision>
-                        <xacro:default_inertial mass="20"/>
-                </link>
-                <joint name="back_${leftright}_wheel_to_back_axle" type="revolute">
+                        <xacro:default_inertial mass="${wheel_mass}"/>
+                </link>
+                <joint name="back_${leftright}_wheel_to_back_axle" type="continuous">
                         <axis xyz="0 0 1" />
                         <limit lower="${lower}" upper="${upper}" effort="1000.0" velocity="1.0"/>
@@ -151,7 +152,7 @@
                 </joint>
                 <gazebo reference="back_${leftright}_wheel">
-                        <mu1 value="200.0"/>
-                        <mu2 value="100.0"/>
-                        <kp value="10000000.0" />
+                        <mu1 value="20.0"/>
+                        <mu2 value="10.0"/>
+                        <kp value="10000.0" />
                         <kd value="1.0" />
                         <material>Gazebo/White</material>
@@ -171,5 +172,5 @@
                                 </geometry>
                         </collision>
-                        <xacro:default_inertial mass="1e-5"/>
+                        <xacro:default_inertial mass="${camera_mass}"/>
                 </link>
                 <joint name="camera_joint" type="fixed">
@@ -222,8 +223,14 @@
         <xacro:car_axle frontback="front" position="1" upper="0.785" lower="-0.785" />
         <xacro:car_axle frontback="back" position="-1" upper="0.785" lower="-0.785" />
+        <!--
         <xacro:car_front_wheel leftright="left" lr="${(axlelength/2) + 0.05}" axle="1"
                 position="1" upper="0.785" lower="-0.393" />
         <xacro:car_front_wheel leftright="right" lr="${-(axlelength/2) - 0.05}" axle="1"
                 position="-1" upper="0.393" lower="-0.785" />
+        -->
+        <xacro:car_front_wheel leftright="left" lr="${(axlelength/2) + 0.05}" axle="1"
+                position="1" upper="3140" lower="-3140" />
+        <xacro:car_front_wheel leftright="right" lr="${-(axlelength/2) - 0.05}" axle="1"
+                position="-1" upper="3140" lower="-3140" />
         <xacro:car_back_wheel leftright="left" lr="${(axlelength/2) + 0.05}" axle="-1"
                 upper="${3.14*1000}" lower="${-3.14*1000}" />
@@ -233,27 +240,25 @@
 -->
         <gazebo>
-                <!--
-        -->
+                <plugin name="gazebo_ros_control" filename="libgazebo_ros_control.so">
+                </plugin>
                 <plugin name="diff_drive_controller" filename="libgazebo_ros_diff_drive.so">
                         <alwaysOn>true</alwaysOn>
                         <commandTopic>cmd_vel</commandTopic>
-                        <leftJoint>front_left_wheel_to_front_axle</leftJoint>
-                        <leftJoint>back_left_wheel_to_back_axle</leftJoint>
-                        <legacyMode>true</legacyMode>
+                        <legacyMode>false</legacyMode>
                         <odometryFrame>odom</odometryFrame>
                         <odometrySource>odom</odometrySource>
                         <odometryTopic>odom</odometryTopic>
-                        <publishTf>false</publishTf>
-                        <publishWheelJointState>false</publishWheelJointState>
-                        <publishWheelTF>false</publishWheelTF>
-                        <rightJoint>front_right_wheel_to_front_axle</rightJoint>
-                        <rightJoint>back_right_wheel_to_back_axle</rightJoint>
+                        <publishTf>true</publishTf>
+                        <publishWheelJointState>true</publishWheelJointState>
+                        <publishWheelTF>true</publishWheelTF>
                         <robotBaseFrame>base_footprint</robotBaseFrame>
                         <rosDebugLevel>na</rosDebugLevel>
-                        <wheelTorque>1</wheelTorque>
+                        <wheelTorque>5</wheelTorque>
                         <updateRate>${update_rate}</updateRate>
                         <wheelAcceleration>20</wheelAcceleration>
                         <wheelDiameter>${wheelradius * 2}</wheelDiameter>
                         <wheelSeparation>${axlelength}</wheelSeparation>
+                        <leftJoint>front_left_wheel_to_front_axle</leftJoint>
+                        <rightJoint>front_right_wheel_to_front_axle</rightJoint>
                 </plugin>
         </gazebo>

Commit message: Gazebo Model Moving With Twist Messages
Friction, Stiffness, and Damping Coefficients Need to Be Corrected

File: src/car_model/urdf/carModel.xacro (robot description, xacro)
@@ -34,5 +34,5 @@
                                         <box size="0.001 0.001 0.001"/>
                                 </geometry>
-                                <origin rpy="0 0 0" xyz="0 0 0"/>
+                                <origin rpy="0 0 0" xyz="0.001 0.001 0.001"/>
                         </visual>
                         <collision>
@@ -116,5 +116,7 @@
                 <joint name="front_${leftright}_wheel_to_front_axle" type="continuous">
                         <axis xyz="0 0 1" />
+                        <!--
                         <limit lower="${lower}" upper="${upper}" effort="1000.0" velocity="1.0"/>
+                        -->
                         <parent link="base_footprint" />
                         <child link="front_${leftright}_wheel" />
@@ -122,7 +124,7 @@
                 </joint>
                 <gazebo reference="front_${leftright}_wheel">
-                        <mu1 value="20.0"/>
-                        <mu2 value="10.0"/>
-                        <kp value="10000.0" />
+                        <mu1 value="200.0"/>
+                        <mu2 value="100.0"/>
+                        <kp value="100000.0" />
                         <kd value="1.0" />
                         <material>Gazebo/White</material>
@@ -146,5 +148,7 @@
                 <joint name="back_${leftright}_wheel_to_back_axle" type="continuous">
                         <axis xyz="0 0 1" />
+                        <!--
                         <limit lower="${lower}" upper="${upper}" effort="1000.0" velocity="1.0"/>
+                        -->
                         <parent link="base_footprint" />
                         <child link="back_${leftright}_wheel" />
@@ -152,7 +156,7 @@
                 </joint>
                 <gazebo reference="back_${leftright}_wheel">
-                        <mu1 value="20.0"/>
-                        <mu2 value="10.0"/>
-                        <kp value="10000.0" />
+                        <mu1 value="200.0"/>
+                        <mu2 value="100.0"/>
+                        <kp value="100000.0" />
                         <kd value="1.0" />
                         <material>Gazebo/White</material>
@@ -247,5 +251,4 @@
                         <legacyMode>false</legacyMode>
                         <odometryFrame>odom</odometryFrame>
-                        <odometrySource>odom</odometrySource>
                         <odometryTopic>odom</odometryTopic>
                         <publishTf>true</publishTf>
@@ -254,7 +257,7 @@
                         <robotBaseFrame>base_footprint</robotBaseFrame>
                         <rosDebugLevel>na</rosDebugLevel>
-                        <wheelTorque>5</wheelTorque>
+                        <wheelTorque>30</wheelTorque>
                         <updateRate>${update_rate}</updateRate>
-                        <wheelAcceleration>20</wheelAcceleration>
+                        <wheelAcceleration>2</wheelAcceleration>
                         <wheelDiameter>${wheelradius * 2}</wheelDiameter>
                         <wheelSeparation>${axlelength}</wheelSeparation>

Commit message: Separated RViz Car Publishing Functionality Into Two Files
car_publisher.py used by the self-driving scripts; twist_driver.py for the default Twist message driving

File: src/car_model/urdf/carModel.xacro (robot description, xacro)
@@ -22,4 +22,11 @@
         <xacro:property name="wheel_mass" value="1e+0" />
         <xacro:property name="camera_mass" value="1e-2" />
+        <xacro:macro name="gazebo_wheel_elements" >
+                <mu1 value="2000.0"/>
+                <mu2 value="2000.0"/>
+                <kp value="1000.0" />
+                <kd value="1.0" />
+                <material>Gazebo/White</material>
+        </xacro:macro>
         <xacro:macro name="default_inertial" params="mass">
                 <inertial>
@@ -114,9 +121,7 @@
                         <xacro:default_inertial mass="${wheel_mass}"/>
                 </link>
-                <joint name="front_${leftright}_wheel_to_front_axle" type="continuous">
-                        <axis xyz="0 0 1" />
-                        <!--
+                <joint name="front_${leftright}_wheel_to_front_axle" type="revolute">
+                        <axis xyz="1 0 0" />
                         <limit lower="${lower}" upper="${upper}" effort="1000.0" velocity="1.0"/>
-                        -->
                         <parent link="base_footprint" />
                         <child link="front_${leftright}_wheel" />
@@ -124,9 +129,5 @@
                 </joint>
                 <gazebo reference="front_${leftright}_wheel">
-                        <mu1 value="200.0"/>
-                        <mu2 value="100.0"/>
-                        <kp value="100000.0" />
-                        <kd value="1.0" />
-                        <material>Gazebo/White</material>
+                        <xacro:gazebo_wheel_elements />
                 </gazebo>
         </xacro:macro>
@@ -156,9 +157,5 @@
                 </joint>
                 <gazebo reference="back_${leftright}_wheel">
-                        <mu1 value="200.0"/>
-                        <mu2 value="100.0"/>
-                        <kp value="100000.0" />
-                        <kd value="1.0" />
-                        <material>Gazebo/White</material>
+                        <xacro:gazebo_wheel_elements />
                 </gazebo>
         </xacro:macro>
@@ -227,14 +224,14 @@
         <xacro:car_axle frontback="front" position="1" upper="0.785" lower="-0.785" />
         <xacro:car_axle frontback="back" position="-1" upper="0.785" lower="-0.785" />
-        <!--
         <xacro:car_front_wheel leftright="left" lr="${(axlelength/2) + 0.05}" axle="1"
                 position="1" upper="0.785" lower="-0.393" />
         <xacro:car_front_wheel leftright="right" lr="${-(axlelength/2) - 0.05}" axle="1"
                 position="-1" upper="0.393" lower="-0.785" />
-        -->
+        <!--
         <xacro:car_front_wheel leftright="left" lr="${(axlelength/2) + 0.05}" axle="1"
                 position="1" upper="3140" lower="-3140" />
         <xacro:car_front_wheel leftright="right" lr="${-(axlelength/2) - 0.05}" axle="1"
                 position="-1" upper="3140" lower="-3140" />
+        -->
         <xacro:car_back_wheel leftright="left" lr="${(axlelength/2) + 0.05}" axle="-1"
                 upper="${3.14*1000}" lower="${-3.14*1000}" />

Commit message: Minor Car_Model Corrections

File: src/car_model/urdf/carModel.xacro (robot description, xacro)
@@ -66,5 +66,5 @@
                 </joint>
         </xacro:macro>
-        <xacro:macro name="car_axle" params="frontback position upper lower">
+        <xacro:macro name="car_axle" params="frontback position">
                <link name="${frontback}_axle">
                        <visual>
@@ -83,5 +83,4 @@
                <joint name="${frontback}_axle_to_base" type="fixed">
                        <axis xyz="1 0 0" />
-                       <limit lower="${lower}" upper="${upper}" effort="1000.0" velocity="1.0"/>
                        <mimic joint="base_footprint_joint" multiplier="1"/>
                        <parent link="base_footprint" />
@@ -160,6 +159,6 @@
         <xacro:car_base />
         <xacro:camera_link height="240" width="320" />
-        <xacro:car_axle frontback="front" position="1" upper="0.785" lower="-0.785" />
-        <xacro:car_axle frontback="back" position="-1" upper="0.785" lower="-0.785" />
+        <xacro:car_axle frontback="front" position="1" />
+        <xacro:car_axle frontback="back" position="-1" />
         <xacro:car_front_wheel leftright="left" lr="${(axlelength/2) + 0.05}" axle="1"
                 position="1" upper="0.785" lower="-0.393" />

File: src/car_model/urdf/gazeboCar.xacro (robot description, xacro)
@@ -18,6 +18,6 @@
         <xacro:property name="axlelength" value="0.4" />
         <xacro:property name="update_rate" value="5.0" />
-        <xacro:property name="base_mass" value="1e-1" />
-        <xacro:property name="axle_mass" value="${0.5*1e-1}" />
+        <xacro:property name="base_mass" value="1e+0" />
+        <xacro:property name="axle_mass" value="1e-1" />
         <xacro:property name="wheel_mass" value="1e+0" />
         <xacro:property name="camera_mass" value="1e-2" />
@@ -48,5 +48,5 @@
                                 </geometry>
                         </collision>
-                        <xacro:default_inertial mass="${base_mass/100}"/>
+                        <xacro:default_inertial mass="${base_mass/1000}"/>
                 </link>
                 <gazebo reference="base_footprint">
@@ -79,5 +79,5 @@
                 </gazebo>
         </xacro:macro>
-        <xacro:macro name="car_axle" params="frontback position upper lower">
+        <xacro:macro name="car_axle" params="frontback position">
                <link name="${frontback}_axle">
                        <visual>
@@ -96,5 +96,4 @@
                <joint name="${frontback}_axle_to_base" type="fixed">
                        <axis xyz="1 0 0" />
-                       <limit lower="${lower}" upper="${upper}" effort="1000.0" velocity="1.0"/>
                        <mimic joint="base_footprint_joint" multiplier="1"/>
                        <parent link="base_footprint" />
@@ -175,10 +174,6 @@
                                 <plugin name="camera_controller" filename="libgazebo_ros_camera.so">
                                         <alwaysOn>true</alwaysOn>
-                                        <updateRate>0.00</updateRate>
+                                        <cameraInfoTopicName>camera_info</cameraInfoTopicName>
                                         <cameraName>car_model_camera</cameraName>
-                                        <imageTopicName>image_raw</imageTopicName>
-                                        <cameraInfoTopicName>camera_info</cameraInfoTopicName>
-                                        <frameName>odom</frameName>
-                                        <hackBaseline>0.07</hackBaseline>
                                         <distortionK1>0.0</distortionK1>
                                         <distortionK2>0.0</distortionK2>
@@ -186,4 +181,9 @@
                                         <distortionT1>0.0</distortionT1>
                                         <distortionT2>0.0</distortionT2>
+                                        <frameName>/odom</frameName>
+                                        <hackBaseline>0.07</hackBaseline>
+                                        <imageTopicName>image_raw</imageTopicName>
+                                        <robotNamespace>car_model</robotNamespace>
+                                        <updateRate>0.00</updateRate>
                                 </plugin>
                         </sensor>
@@ -193,6 +193,6 @@
         <xacro:car_base />
         <xacro:camera_link height="240" width="320" />
-        <xacro:car_axle frontback="front" position="1" upper="0.785" lower="-0.785" />
-        <xacro:car_axle frontback="back" position="-1" upper="0.785" lower="-0.785" />
+        <xacro:car_axle frontback="front" position="1" />
+        <xacro:car_axle frontback="back" position="-1" />
         <xacro:car_wheel frontback="front" leftright="left" fb="0.3" lr="${(axlelength/2) + 0.05}" />
         <xacro:car_wheel frontback="front" leftright="right" fb="0.3" lr="${-(axlelength/2) - 0.05}" />
@@ -202,23 +202,25 @@
                 <plugin name="skid_steer_drive_controller" filename="libgazebo_ros_skid_steer_drive.so">
                         <broadcastTF>true</broadcastTF>
-                        <commandTopic>cmd_vel</commandTopic>
+                        <commandTopic>/cmd_vel</commandTopic>
                         <covariance_x>0.000100</covariance_x>
                         <covariance_y>0.000100</covariance_y>
-                        <covariance_yaw>0.010000</covariance_yaw>
+                        <covariance_yaw>1.57</covariance_yaw>
                         <leftFrontJoint>front_left_wheel_to_front_axle</leftFrontJoint>
                         <leftRearJoint>back_left_wheel_to_back_axle</leftRearJoint>
                         <odometryFrame>odom</odometryFrame>
-                        <odometryTopic>odom</odometryTopic>
+                        <odometryTopic>/odom</odometryTopic>
                         <rightFrontJoint>front_right_wheel_to_front_axle</rightFrontJoint>
                         <rightRearJoint>back_right_wheel_to_back_axle</rightRearJoint>
                         <robotBaseFrame>base_footprint</robotBaseFrame>
-                        <robotNamespace>/</robotNamespace>
-                        <topicName>cmd_vel</topicName>
-                        <torque>18</torque>
+                        <robotNamespace>car_model</robotNamespace>
+                        <topicName>/cmd_vel</topicName>
+                        <torque>20</torque>
                         <updateRate>100.0</updateRate>
                         <wheelDiameter>${wheelradius * 2}</wheelDiameter>
                         <wheelSeparation>${axlelength}</wheelSeparation>
                 </plugin>
-                <plugin name="gazebo_ros_control" filename="libgazebo_ros_control.so" />
+                <plugin name="gazebo_ros_control" filename="libgazebo_ros_control.so">
+                        <robotNamespace>car_model</robotNamespace>
+                </plugin>
         </gazebo>
 </robot>
